Commit message: fix xacro file

File: src/magni_description/urdf/magni.transmission.xacro (robot description, xacro)
@@ -4,11 +4,11 @@
     <hardware>
         <plugin>ubiquity_motor_ros2/MotorHardware</plugin>
-    <hardware>
-    <joint name="$left_wheel_joint">
+    </hardware>
+    <joint name="left_wheel_joint">
         <command_interface name="velocity"/>
         <state_interface name="position"/>
         <state_interface name="effort"/>
-      </joint>
-    <joint name="$right_wheel_joint">
+    </joint>
+    <joint name="right_wheel_joint">
         <command_interface name="velocity"/>
         <state_interface name="position"/>
