Commit message: fix caster wheels

File: src/magni_description/urdf/magni.urdf.xacro (robot description, xacro)
@@ -27,16 +27,4 @@
       </geometry>
     </visual>
-	  <visual>
-      <origin xyz="${-wheel_xpos-0.169} 0.17 ${-wheel_r+0.09}" rpy="0 0 ${pi}" />
-      <geometry>
-        <mesh filename="package://magni_description/meshes/caster_wheel.dae" />
-      </geometry>
-    </visual>
-	  <visual>
-      <origin xyz="${-wheel_xpos-0.169} -0.17 ${-wheel_r+0.09}" rpy="0 0 ${pi}" />
-      <geometry>
-        <mesh filename="package://magni_description/meshes/caster_wheel.dae" />
-      </geometry>
-    </visual>
     <collision>
 	    <origin xyz="${-wheel_xpos} 0 ${-wheel_r+0.151}" rpy="0 0 0" />
@@ -49,16 +37,4 @@
       <geometry>
         <box size="0.375 0.268 0.034"/>
-      </geometry>
-    </collision>
-    <collision>
-      <origin xyz="${-wheel_xpos-0.169} 0.169 ${-wheel_r+0.106}" rpy="0 0 0" />
-      <geometry>
-        <box size="0.1 0.07 0.07"/>
-      </geometry>
-    </collision>
-    <collision>
-      <origin xyz="${-wheel_xpos-0.169} -0.169 ${-wheel_r+0.106}" rpy="0 0 0" />
-      <geometry>
-        <box size="0.1 0.07 0.07"/>
       </geometry>
     </collision>
@@ -170,15 +146,45 @@
   <!-- Macro for defining caster wheels -->
   <xacro:macro name="caster_wheel" params="prefix reflect">
+    <link name="${prefix}_caster_wheel_support">
+      <collision>
+        <origin xyz="-0.025 ${reflect*0.01} 0" rpy="0 0 0" />
+        <geometry>
+           <box size="0.05 0.04 0.01"/>
+        </geometry>
+      </collision>
+      <visual>
+        <origin xyz="0 0 0" rpy="0 0 ${pi}" />
+        <geometry>
+          <mesh filename="package://magni_description/meshes/caster_wheel.dae" />
+        </geometry>
+      </visual>
+      <xacro:box_inertial_with_origin  x="0.05" y="0.04" z="0.01" mass="0.25">
+        <origin xyz="-0.025 ${reflect*0.01} 0" rpy="0 0 0" />
+      </xacro:box_inertial_with_origin>
+    </link>
+    <joint name="${prefix}_caster_wheel_support_joint" type="continuous">
+      <origin xyz="${-wheel_xpos-0.169} ${reflect*0.169} ${-wheel_r+0.09}" rpy="0 0 0" />
+      <axis xyz="0 0 1" rpy="0 0 0" />
+      <parent link="base_link"/>
+      <child link="${prefix}_caster_wheel_support"/>
+      <dynamics damping="0.0" friction="0.0"/>
+    </joint>
     <link name="${prefix}_caster_wheel">
       <collision>
-        <origin xyz="${-wheel_xpos-0.19} ${reflect*0.169} ${-wheel_r+0.04}" rpy="0 0 0" />
-        <geometry>
-          <sphere radius="0.04"/>
-        </geometry>
-      </collision>
+        <origin xyz="0 0 0" rpy="0 ${pi/2} 0" />
+        <geometry>
+          <cylinder length="0.02" radius="0.0381"/>
+        </geometry>
+      </collision>
+      <xacro:cylinder_inertial_with_origin radius="0.0381" length="0.02" mass="0.25">
+        <origin xyz="0 0 0" rpy="0 ${pi/2} 0" />
+      </xacro:cylinder_inertial_with_origin>
     </link>
     <joint name="${prefix}_caster_wheel_joint" type="continuous">
-      <parent link="base_link"/>
+      <origin xyz="-0.02 0 -0.053" rpy="0 0 ${pi/2}" />
+      <axis xyz="1 0 0" rpy="0 0 0" />
+      <parent link="${prefix}_caster_wheel_support"/>
       <child link="${prefix}_caster_wheel"/>
+      <dynamics damping="0.0" friction="0.0"/>
     </joint>
   </xacro:macro>

Commit message: create bringup package for real robot and fix simulation

File: src/magni_description/urdf/magni.urdf.xacro (robot description, xacro)
@@ -147,10 +147,4 @@
   <xacro:macro name="caster_wheel" params="prefix reflect">
     <link name="${prefix}_caster_wheel_support">
-      <collision>
-        <origin xyz="-0.025 ${reflect*0.01} 0" rpy="0 0 0" />
-        <geometry>
-           <box size="0.05 0.04 0.01"/>
-        </geometry>
-      </collision>
       <visual>
         <origin xyz="0 0 0" rpy="0 0 ${pi}" />
@@ -159,7 +153,4 @@
         </geometry>
       </visual>
-      <xacro:box_inertial_with_origin  x="0.05" y="0.04" z="0.01" mass="0.25">
-        <origin xyz="-0.025 ${reflect*0.01} 0" rpy="0 0 0" />
-      </xacro:box_inertial_with_origin>
     </link>
     <joint name="${prefix}_caster_wheel_support_joint" type="continuous">

Commit message: working on brinup package and ensure teleop joy is working

File: src/magni_description/urdf/magni.urdf.xacro (robot description, xacro)
@@ -153,4 +153,9 @@
         </geometry>
       </visual>
+      <collision>
+        <geometry>
+          <box size="0.03 0.03 0.003" />
+        </geometry>
+      </collision>
     </link>
     <joint name="${prefix}_caster_wheel_support_joint" type="continuous">

Commit message: work in progress

File: src/magni_description/urdf/magni.urdf.xacro (robot description, xacro)
@@ -107,6 +107,6 @@
   </link>
   <joint name="base_footprint_joint" type="fixed">
-    <parent link="base_footprint"/>
-    <child link="base_link"/>
+    <parent link="base_link"/>
+    <child link="base_footprint"/>
     <origin xyz="0 0 ${wheel_r}" rpy="0 0 0"/>
   </joint>

File: src/magni_description/urdf/sensors/raspi_camera.xacro (robot description, xacro)
@@ -31,5 +31,5 @@
     </joint>
     <gazebo reference="${name}_sensor">
-      <sensor type="camera" name="camera1">
+      <sensor type="camera" name="${name}">
         <update_rate>30.0</update_rate>
         <camera name="raspi_camera">

File: src/magni_description/urdf/sensors/sonar_hc-sr04.xacro (robot description, xacro)
@@ -51,5 +51,5 @@
         </ray>
         <!-- Gazebo-ROS interface plugin -->
-        <plugin filename="libgazebo_ros_range.so" name="gazebo_ros_range">
+        <!-- <plugin filename="libgazebo_ros_range.so" name="gazebo_ros_range">
           <gaussianNoise>0.015</gaussianNoise>
           <alwaysOn>true</alwaysOn>
@@ -59,5 +59,5 @@
           <fov>0.5</fov>
           <radiation>ultrasound</radiation>
-        </plugin>
+        </plugin> -->
       </sensor>
     </gazebo>

File: src/magni_description/urdf/sensors/ur50_lidar.xacro (robot description, xacro)
@@ -54,8 +54,8 @@
       </ray>
       <!--<plugin name="gazebo_ros_head_hokuyo_controller" filename="libgazebo_ros_gpu_laser.so">-->
-      <plugin name="gazebo_ros_head_hokuyo_controller" filename="libgazebo_ros_laser.so">
+      <!-- <plugin name="gazebo_ros_head_hokuyo_controller" filename="libgazebo_ros_laser.so">
         <topicName>/scan</topicName>
         <frameName>${name}</frameName>
-      </plugin>
+      </plugin> -->
     </sensor>
   </gazebo>

File: src/magni_description/urdf/sensors/ur_c1_lidar.xacro (robot description, xacro)
@@ -54,8 +54,8 @@
       </ray>
       <!--<plugin name="gazebo_ros_head_hokuyo_controller" filename="libgazebo_ros_gpu_laser.so">-->
-      <plugin name="gazebo_ros_head_hokuyo_controller" filename="libgazebo_ros_laser.so">
+      <!-- <plugin name="gazebo_ros_head_hokuyo_controller" filename="libgazebo_ros_laser.so">
         <topicName>/scan</topicName>
         <frameName>${name}</frameName>
-      </plugin>
+      </plugin> -->
     </sensor>
   </gazebo>

File: src/magni_webots/resource/magni_wb.urdf.xacro (robot description, xacro)
@@ -2,5 +2,5 @@
 <robot name="magni" xmlns:xacro="http://wiki.ros.org/xacro">
     <webots>
-        <device reference="camera1" type="Camera">
+        <device reference="raspicam" type="Camera">
             <ros>
                 <topicName>/rpicam</topicName>
@@ -9,8 +9,11 @@
             </ros>
         </device>
-        <device reference="laser" type="Ray">
+        <device reference="laser" type="Lidar">
             <ros>
+                <enabled>true</enabled>
+                <updateRate>10</updateRate>
                 <topicName>/scan</topicName>
                 <alwaysOn>true</alwaysOn>
+                <frameName>laser</frameName>
             </ros>
         </device>

Commit message: complete cartographer implementation

File: src/magni_description/urdf/magni.urdf.xacro (robot description, xacro)
@@ -107,6 +107,6 @@
   </link>
   <joint name="base_footprint_joint" type="fixed">
-    <parent link="base_link"/>
-    <child link="base_footprint"/>
+    <parent link="base_footprint"/>
+    <child link="base_link"/>
     <origin xyz="0 0 ${wheel_r}" rpy="0 0 0"/>
   </joint>
