Commit message: fix simulation frames

File: src/magni_description/urdf/magni.control.xacro (robot description, xacro)
@@ -25,4 +25,8 @@
             <state_interface name="effort"/>
         </joint>
+        <joint name="left_caster_wheel_joint"/>
+        <joint name="right_caster_wheel_joint"/>
+        <joint name="left_caster_wheel_base_joint"/>
+        <joint name="right_caster_wheel_base_joint"/>
     </ros2_control>
 </xacro:macro>

File: src/magni_description/urdf/magni.urdf.xacro (robot description, xacro)
@@ -39,73 +39,74 @@
       </geometry>
     </collision>
+    <xacro:if value="${tower_installed}">
+      <!-- Robot Tower -->
+      <visual>
+        <origin xyz="0 0 0.005" rpy="0 0 0" />
+        <geometry>
+          <mesh filename="package://magni_description/meshes/magni_tower.dae" />
+        </geometry>
+      </visual>
+      <!-- Collision for screen -->
+      <collision>
+        <origin xyz="0.115 0 0.635" rpy="0 0.56 0" />
+        <geometry>
+          <box size="0.04 0.23 0.15"/>
+        </geometry>
+      </collision>
+      <!-- Collision for tower vertical-->
+      <collision>
+        <origin xyz="0.08 0 0.37" rpy="0 0 0" />
+        <geometry>
+          <box size="0.06 0.24 0.40"/>
+        </geometry>
+      </collision>
+      <!-- Collision for tower horizontal -->
+      <collision>
+        <origin xyz="-0.1 0 0.18" rpy="0 0 0" />
+        <geometry>
+          <box size="0.42 0.24 0.03"/>
+        </geometry>
+      </collision>
+      <!-- Lower shelf -->
+      <collision>
+        <origin xyz="-0.18 0 0.2" rpy="0 0 0" />
+        <geometry>
+          <box size="0.35 0.408 0.005"/>
+        </geometry>
+      </collision>
+      <!-- Upper shelf -->
+      <collision>
+        <origin xyz="-0.1 0 0.53" rpy="0 0 0" />
+        <geometry>
+          <box size="0.32 0.42 0.02"/>
+        </geometry>
+      </collision>
+    </xacro:if>
+    <xacro:if value="${shell_installed}">
+      <!-- Robot shell -->
+      <visual>
+        <origin xyz="0 0 0.005" rpy="0 0 0" />
+        <geometry>
+          <mesh filename="package://magni_description/meshes/magni_shell.dae" />
+        </geometry>
+      </visual>
+      <!-- Collision for shell -->
+      <collision>
+        <origin xyz="-0.175 0 0.07" rpy="0 0.0 0" />
+        <geometry>
+          <box size="0.3 0.33 0.2"/>
+        </geometry>
+      </collision>
+    </xacro:if>
+  </link>
+<!-- Fixed offset from the floor to the center of the wheels -->
+  <link name="base_footprint">
     <xacro:box_inertial_with_origin  x="0.398" y="0.221" z="0.150" mass="10.0">
       <origin xyz="-0.15 0 0.03" rpy="0 0 0" />
     </xacro:box_inertial_with_origin>
-    <xacro:if value="${tower_installed}">
-      <!-- Robot Tower -->
-      <visual>
-        <origin xyz="0 0 0.005" rpy="0 0 0" />
-        <geometry>
-          <mesh filename="package://magni_description/meshes/magni_tower.dae" />
-        </geometry>
-      </visual>
-      <!-- Collision for screen -->
-      <collision>
-        <origin xyz="0.115 0 0.635" rpy="0 0.56 0" />
-        <geometry>
-          <box size="0.04 0.23 0.15"/>
-        </geometry>
-      </collision>
-      <!-- Collision for tower vertical-->
-      <collision>
-        <origin xyz="0.08 0 0.37" rpy="0 0 0" />
-        <geometry>
-          <box size="0.06 0.24 0.40"/>
-        </geometry>
-      </collision>
-      <!-- Collision for tower horizontal -->
-      <collision>
-        <origin xyz="-0.1 0 0.18" rpy="0 0 0" />
-        <geometry>
-          <box size="0.42 0.24 0.03"/>
-        </geometry>
-      </collision>
-      <!-- Lower shelf -->
-      <collision>
-        <origin xyz="-0.18 0 0.2" rpy="0 0 0" />
-        <geometry>
-          <box size="0.35 0.408 0.005"/>
-        </geometry>
-      </collision>
-      <!-- Upper shelf -->
-      <collision>
-        <origin xyz="-0.1 0 0.53" rpy="0 0 0" />
-        <geometry>
-          <box size="0.32 0.42 0.02"/>
-        </geometry>
-      </collision>
-    </xacro:if>
-    <xacro:if value="${shell_installed}">
-      <!-- Robot shell -->
-      <visual>
-        <origin xyz="0 0 0.005" rpy="0 0 0" />
-        <geometry>
-          <mesh filename="package://magni_description/meshes/magni_shell.dae" />
-        </geometry>
-      </visual>
-      <!-- Collision for shell -->
-      <collision>
-        <origin xyz="-0.175 0 0.07" rpy="0 0.0 0" />
-        <geometry>
-          <box size="0.3 0.33 0.2"/>
-        </geometry>
-      </collision>
-    </xacro:if>
   </link>
-  <!-- Fixed offset from the floor to the center of the wheels -->
-  <link name="base_footprint"/>
   <joint name="base_footprint_joint" type="fixed">
-    <parent link="base_link"/>
-    <child link="base_footprint"/>
+    <parent link="base_footprint"/>
+    <child link="base_link"/>
     <origin xyz="0 0 ${wheel_r}" rpy="0 0 0"/>
   </joint>
@@ -146,23 +147,44 @@
   <!-- Macro for defining caster wheels -->
   <xacro:macro name="caster_wheel" params="prefix reflect">
-    <link name="${prefix}_caster_wheel_support">
-      <visual>
-        <origin xyz="0 0 0" rpy="0 0 ${pi}" />
-        <geometry>
-          <mesh filename="package://magni_description/meshes/caster_wheel.dae" />
-        </geometry>
-      </visual>
-      <collision>
+    <link name="${prefix}_caster_wheel_base">
+      <visual>
+        <origin xyz="0 0 0" rpy="0 0 0" />
         <geometry>
           <box size="0.03 0.03 0.003" />
         </geometry>
-      </collision>
-    </link>
-    <joint name="${prefix}_caster_wheel_support_joint" type="continuous">
+      </visual>
+      <collision>
+        <geometry>
+          <box size="0.03 0.03 0.003" />
+        </geometry>
+      </collision>
+    </link>
+    <joint name="${prefix}_caster_wheel_base_joint" type="continuous">
       <origin xyz="${-wheel_xpos-0.169} ${reflect*0.169} ${-wheel_r+0.09}" rpy="0 0 0" />
       <axis xyz="0 0 1" rpy="0 0 0" />
       <parent link="base_link"/>
+      <child link="${prefix}_caster_wheel_base"/>
+      <dynamics damping="0.0" friction="0.0"/>
+    </joint>
+    <link name="${prefix}_caster_wheel_support">
+      <visual>
+        <origin xyz="0 0 0" rpy="0 0 ${pi}" />
+        <geometry>
+          <mesh filename="package://magni_description/meshes/caster_wheel.dae" />
+        </geometry>
+      </visual>
+      <collision>
+        <geometry>
+          <box size="0.03 0.003 0.03" />
+        </geometry>
+      </collision>
+      <xacro:box_inertial_with_origin  x="0.03" y="0.003" z="0.03" mass="0.1">
+        <origin xyz="0 0 0" rpy="0 0 0" />
+      </xacro:box_inertial_with_origin>
+    </link>
+    <joint name="${prefix}_caster_wheel_support_joint" type="fixed">
+      <origin xyz="0 0 0" rpy="0 0 0" />
+      <parent link="${prefix}_caster_wheel_base"/>
       <child link="${prefix}_caster_wheel_support"/>
-      <dynamics damping="0.0" friction="0.0"/>
     </joint>
     <link name="${prefix}_caster_wheel">

File: src/magni_description/urdf/sensors/ur50_lidar.xacro (robot description, xacro)
@@ -25,5 +25,5 @@
   <gazebo reference="${name}">
     <!--<sensor type="gpu_ray" name="${name}_sensor>-->
-    <sensor type="ray" name="${name}_sensor">
+    <sensor type="ray" name="${name}">
       <pose>0 0 0 0 0 0</pose>
       <visualize>false</visualize>

File: src/magni_description/urdf/sensors/ur_c1_lidar.xacro (robot description, xacro)
@@ -25,5 +25,5 @@
   <gazebo reference="${name}">
     <!--<sensor type="gpu_ray" name="${name}_sensor>-->
-    <sensor type="ray" name="${name}_sensor">
+    <sensor type="ray" name="${name}">
       <pose>0 0 0 0 0 0</pose>
       <visualize>false</visualize>

File: src/magni_webots/resource/magni_wb.urdf.xacro (robot description, xacro)
@@ -9,5 +9,5 @@
             </ros>
         </device>
-        <device reference="laser_sensor" type="Ray">
+        <device reference="laser" type="Ray">
             <ros>
                 <topicName>/scan</topicName>

Commit message: fix ros control bad usage

File: src/magni_description/urdf/magni.control.xacro (robot description, xacro)
@@ -25,8 +25,4 @@
             <state_interface name="effort"/>
         </joint>
-        <joint name="left_caster_wheel_joint"/>
-        <joint name="right_caster_wheel_joint"/>
-        <joint name="left_caster_wheel_base_joint"/>
-        <joint name="right_caster_wheel_base_joint"/>
     </ros2_control>
 </xacro:macro>
